Commit message: Add mock and sim hardware interface option

File: fairino20_v6_moveit2_config/config/fairino20_v6_robot.ros2_control.xacro (robot description, xacro)
@@ -1,10 +1,14 @@
 <?xml version="1.0"?>
 <robot xmlns:xacro="http://www.ros.org/wiki/xacro">
-    <xacro:macro name="fairino20_v6_robot_ros2_control" params="name initial_positions_file">
+    <xacro:macro name="fairino20_v6_robot_ros2_control" params="name initial_positions_file use_mock_hardware">
         <xacro:property name="initial_positions" value="${load_yaml(initial_positions_file)['initial_positions']}"/>
         <ros2_control name="${name}" type="system">
             <hardware>
-                <!-- By default, set up controllers for simulation. This won't work on real hardware -->
-                <plugin>mock_components/GenericSystem</plugin>
+                <xacro:if value="${use_mock_hardware}">
+                    <plugin>mock_components/GenericSystem</plugin>
+                </xacro:if>
+                <xacro:unless value="${use_mock_hardware}">
+                    <plugin>fairino_hardware/FairinoHardwareInterface</plugin>
+                </xacro:unless>
             </hardware>
             <joint name="j1">

File: fairino20_v6_moveit2_config/config/fairino20_v6_robot.urdf.xacro (robot description, xacro)
@@ -2,8 +2,12 @@
 <robot xmlns:xacro="http://www.ros.org/wiki/xacro" name="fairino20_v6_robot">
     <xacro:arg name="initial_positions_file" default="initial_positions.yaml" />
+    <xacro:arg name="use_mock_hardware" default="false" />
     <!-- Import fairino20_v6_robot urdf file -->
     <xacro:include filename="$(find fairino_description)/urdf/fairino20_v6.urdf" />
-    <!-- Import control_xacro -->
+    <!-- Import ros2_control configuration -->
     <xacro:include filename="fairino20_v6_robot.ros2_control.xacro" />
-    <xacro:fairino20_v6_robot_ros2_control name="FakeSystem" initial_positions_file="$(arg initial_positions_file)"/>
+    <xacro:fairino20_v6_robot_ros2_control
+        name="FairinoSystem"
+        initial_positions_file="$(arg initial_positions_file)"
+        use_mock_hardware="$(arg use_mock_hardware)" />
 </robot>
