Commit message: Use the FAIRINO TCP frame, faster plan mode and a simpler operator UI
- fairino_description: fixed frame "flange" (wrist3_link + 120 mm along z),
  measured against the controller FK; servo, planner, gizmo and benchmark
  use it (live difference to tl_cur_pos 0.011 mm / 0.0004 deg)
- RobotStatus: tool_number, user_frame_number, flange_pose, tcp_pose;
  the Viser Status tab compares the Viser and FAIRINO TCP
- roboplan.yaml: TOPP-RA acceleration 1.0 -> 9.4248 rad/s^2 (540 deg/s^2,
  the controller's own MoveJ peak); servo: 2.0 m/s Cartesian limit,
  filter tau 0.03 s
- Viser UI: translucent preview of a planned trajectory before Execute,
  measured TCP axes, plane handles on the gizmo, Home button, buttons
  Enable Servo / Servo Hold / Plan Mode, one Recover button (recover or
  reset_fault as required); no mode switch, no Replay button
- docs: frames, plan-mode acceleration measurements, operator guide,
  tests T33-T38

Co-Authored-By: Claude Opus 5.5 <noreply@anthropic.com>

File: fairino_description/urdf/fairino20_v6.urdf (robot description, URDF)
Before this commit: robot fairino20_v6_robot, 7 links, 6 joints
Links:
- added link flange
Joints:
- added joint flange_joint: type fixed, parent wrist3_link, child flange, origin xyz=0 0 0.12 rpy=0 0 0

File: fairinoplan_bringup/config/fairino20_v6_servo_collision.urdf (robot description, URDF)
Before this commit: robot fairino20_v6_robot, 7 links, 6 joints
Links:
- added link flange
Joints:
- added joint flange_joint: type fixed, parent wrist3_link, child flange, origin xyz=0 0 0.12 rpy=0 0 0
